Commit message: add 传感器仿真

File: src/robot_description/urdf/NaviRobot/NaviRobot.urdf.xacro (robot description, xacro)
@@ -7,7 +7,21 @@
 <xacro:include filename="$(find robot_description)/urdf/NaviRobot/sensor/camera.urdf.xacro"/>
 <xacro:include filename="$(find robot_description)/urdf/NaviRobot/sensor/laser.urdf.xacro"/>
+<!-- 执行器部分 -->
+<xacro:include filename="$(find robot_description)/urdf/NaviRobot/actuator/wheel.urdf.xacro"/>
+<xacro:include filename="$(find robot_description)/urdf/NaviRobot/actuator/caster.urdf.xacro"/>
+<!-- 插件 -->
+<!-- <xacro:include filename="$(find robot_description)/urdf/NaviRobot/plugins/gazebo_control_plugin.xacro"/> -->
+<xacro:include filename="$(find robot_description)/urdf/NaviRobot/plugins/gazebo_sensor_plugin.xacro"/>
+<xacro:include filename="$(find robot_description)/urdf/NaviRobot/NaviRobot.ros2_control.xacro"/>
 <xacro:base_xacro length="0.12" radius="0.10"/>
 <xacro:imu_xacro xyz="0.0 0.0 0.02"/>
 <xacro:camera_xacro xyz="0.10 0.0 0.075"/>
 <xacro:laser_xacro xyz="0.0 0.0 0.10"/>
+<xacro:wheel_xacro wheel_name="left_wheel" xyz="0.0 0.10 -0.06"/>
+<xacro:wheel_xacro wheel_name="right_wheel" xyz="0.0 -0.10 -0.06"/>
+<xacro:caster_xacro caster_name="front_wheel" xyz="0.08 0.0 -0.076"/>
+<xacro:caster_xacro caster_name="back_wheel" xyz="-0.08 0.0 -0.076"/>
+<!-- <xacro:gazebo_control_plugin /> -->
+<xacro:gazebo_sensor_plugin />
+<xacro:NaviRbot_ros2_control />
 </robot>

File: src/robot_description/urdf/NaviRobot/base.urdf.xacro (robot description, xacro)
@@ -1,17 +1,34 @@
 <?xml version="1.0"?>
 <robot xmlns:xacro="http://www.ros.org/wiki/xacro">
-  <!-- ========== 机器人主体 ========== -->
-  <xacro:macro name="base_xacro" params="length radius">
-    <link name="base_link">
-        <!-- 视觉属性 -->
-        <visual>
-        <geometry>
-            <cylinder radius="${radius}" length="${length}"/>
-        </geometry>
-        <material name="white">
-            <color rgba="1.0 1.0 1.0 0.5"/>
-        </material>
-        </visual>
-    </link>
-  </xacro:macro>
+    <xacro:include filename="$(find robot_description)/urdf/NaviRobot/common_inertia.xacro"/>
+    <!-- ========== 机器人主体 ========== -->
+    <xacro:macro name="base_xacro" params="length radius">
+        <link name="base_footprint"/>
+        <link name="base_link">
+            <!-- 视觉属性 -->
+            <visual>
+                <geometry>
+                    <cylinder radius="${radius}" length="${length}"/>
+                </geometry>
+                <material name="white">
+                    <color rgba="1.0 1.0 1.0 0.5"/>
+                </material>
+            </visual>
+            <!-- 碰撞特性 -->
+            <collision>
+                <geometry>
+                    <cylinder radius="${radius}" length="${length}"/>
+                </geometry>
+                <material name="white">
+                    <color rgba="1.0 1.0 1.0 0.5"/>
+                </material>
+            </collision>
+            <xacro:cylinder_inertia m="1.0" r="${radius}" h="${length}"/>
+        </link>
+        <joint name="joint_name" type="fixed">
+            <origin xyz="0.0 0.0 ${length/2+0.032-0.001}" rpy="0.0 0.0 0.0"/>
+            <parent link="base_footprint"/>
+            <child link="base_link"/>
+        </joint>
+    </xacro:macro>
 </robot>

File: src/robot_description/urdf/NaviRobot/sensor/camera.urdf.xacro (robot description, xacro)
@@ -1,23 +1,43 @@
 <?xml version="1.0"?>
 <robot xmlns:xacro="http://www.ros.org/wiki/xacro">
+  <xacro:include filename="$(find robot_description)/urdf/NaviRobot/common_inertia.xacro"/>
   <!-- ========== camera传感器 ========== -->
   <xacro:macro name="camera_xacro" params="xyz">
-    <link name="camera_link">
-        <visual>
-        <geometry>
-            <box size="0.02 0.10 0.02"/>
-        </geometry>
-        <material name="black">
-            <color rgba="0.0 0.0 0.0 0.5"/>
-        </material>
-        </visual>
-    </link>
-    <!-- ========== 固定camera到机器人顶部 ========== -->
-    <joint name="camera_joint" type="fixed">
-        <parent link="base_link"/>
-        <child link="camera_link"/>
-        <!-- 位置：机器人顶部中心 (0.5/2 + 0.05/2 = 0.275) -->
-        <origin xyz="${xyz}" rpy="0.0 0.0 0.0"/>
-    </joint>
+      <link name="camera_link">
+          <visual>
+            <geometry>
+                <box size="0.02 0.10 0.02"/>
+            </geometry>
+            <material name="black">
+                <color rgba="0.0 0.0 0.0 0.5"/>
+            </material>
+          </visual>
+          <!-- 碰撞特性 -->
+          <collision>
+            <geometry>
+                <box size="0.02 0.10 0.02"/>
+            </geometry>
+            <material name="black">
+                <color rgba="0.0 0.0 0.0 0.5"/>
+            </material>
+          </collision>
+          <xacro:box_inertia m="0.01" w="0.02" h="0.10" d="0.02" />
+      </link>
+       <link name="camera_optical_link"></link>
+      <!-- ========== 固定camera到机器人顶部 ========== -->
+      <joint name="camera_joint" type="fixed">
+          <parent link="base_link"/>
+          <child link="camera_link"/>
+          <!-- 位置：机器人顶部中心 (0.5/2 + 0.05/2 = 0.275) -->
+          <origin xyz="${xyz}" rpy="0.0 0.0 0.0"/>
+      </joint>
+      <joint name="camera_optical_joint" type="fixed">
+          <parent link="camera_link" />
+          <child link="camera_optical_link" />
+          <origin xyz="0 0 0" rpy="${-pi/2} 0 ${-pi/2}" />
+      </joint>
+      <gazebo reference="camera_link">
+            <material>Gazebo/Black</material>
+      </gazebo>
   </xacro:macro>
 </robot>

File: src/robot_description/urdf/NaviRobot/sensor/imu.urdf.xacro (robot description, xacro)
@@ -1,15 +1,26 @@
 <?xml version="1.0"?>
 <robot xmlns:xacro="http://www.ros.org/wiki/xacro">
+  <xacro:include filename="$(find robot_description)/urdf/NaviRobot/common_inertia.xacro"/>
   <!-- ========== IMU传感器 ========== -->
   <xacro:macro name="imu_xacro" params="xyz">
     <link name="imu_link">
         <visual>
-        <geometry>
-            <box size="0.02 0.02 0.02"/>
-        </geometry>
-        <material name="black">
-            <color rgba="0.0 0.0 0.0 0.5"/>
-        </material>
+          <geometry>
+              <box size="0.02 0.02 0.02"/>
+          </geometry>
+          <material name="black">
+              <color rgba="0.0 0.0 0.0 0.5"/>
+          </material>
         </visual>
+        <!-- 碰撞特性 -->
+        <collision>
+          <geometry>
+              <box size="0.02 0.02 0.02"/>
+          </geometry>
+          <material name="black">
+              <color rgba="0.0 0.0 0.0 0.5"/>
+          </material>
+        </collision>
+        <xacro:box_inertia m="0.01" w="0.02" d="0.02" h="0.02"/>
     </link>
     <!-- ========== 固定IMU到机器人顶部 ========== -->
@@ -19,4 +30,7 @@
         <origin xyz="${xyz}" rpy="0.0 0.0 0.0"/>
     </joint>
+      <gazebo reference="imu_link">
+            <material>Gazebo/Black</material>
+      </gazebo>
   </xacro:macro>
 </robot>

File: src/robot_description/urdf/NaviRobot/sensor/laser.urdf.xacro (robot description, xacro)
@@ -1,42 +1,69 @@
 <?xml version="1.0"?>
 <robot xmlns:xacro="http://www.ros.org/wiki/xacro">
-  <!-- ========== laser 传感器 ========== -->
-  <xacro:macro name="laser_xacro" params="xyz">
-    <!-- 雷达支撑杆 -->
-    <link name="laser_cylinder_link">
-        <visual>
-        <geometry>
-            <cylinder radius="0.01" length="0.1"/>
-        </geometry>
-        <material name="black">
-            <color rgba="0.0 0.0 0.0 1.0"/>
-        </material>
-        </visual>
-    </link>
-    <!-- 雷达 -->
-    <link name="laser_link">
-        <visual>
-        <geometry>
-            <cylinder radius="0.02" length="0.02"/>
-        </geometry>
-        <material name="black">
-            <color rgba="0.0 0.0 0.0 1.0"/>
-        </material>
-        </visual>
-    </link>
-    <!-- ========== 固定laser支撑杆上 ========== -->
-    <joint name="laser_joint" type="fixed">
-        <parent link="laser_cylinder_link"/>
-        <child link="laser_link"/>
-        <!-- 位置：机器人顶部中心 (0.5/2 + 0.05/2 = 0.275) -->
-        <origin xyz="0.0 0.0 0.05" rpy="0.0 0.0 0.0"/>
-    </joint>
-    <!-- ========== 固定laser支撑杆到机器人顶部 ========== -->
-    <joint name="laser_cylinder_joint" type="fixed">
-        <parent link="base_link"/>
-        <child link="laser_cylinder_link"/>
-        <!-- 位置：机器人顶部中心 (0.5/2 + 0.05/2 = 0.275) -->
-        <origin xyz="${xyz}" rpy="0.0 0.0 0.0"/>
-    </joint>
-  </xacro:macro>
+    <xacro:include filename="$(find robot_description)/urdf/NaviRobot/common_inertia.xacro"/>
+    <!-- ========== laser 传感器 ========== -->
+    <xacro:macro name="laser_xacro" params="xyz">
+        <!-- 雷达支撑杆 -->
+        <link name="laser_cylinder_link">
+            <visual>
+            <geometry>
+                <cylinder radius="0.01" length="0.1"/>
+            </geometry>
+            <material name="black">
+                <color rgba="0.0 0.0 0.0 1.0"/>
+            </material>
+            </visual>
+            <!-- 碰撞特性 -->
+            <collision>
+                <geometry>
+                    <cylinder radius="0.01" length="0.1"/>
+                </geometry>
+                <material name="black">
+                    <color rgba="0.0 0.0 0.0 1.0"/>
+                </material>
+            </collision>
+            <xacro:cylinder_inertia m="0.01" r="0.01" h="0.10" />
+        </link>
+        <!-- 雷达 -->
+        <link name="laser_link">
+            <visual>
+                <geometry>
+                    <cylinder radius="0.02" length="0.02"/>
+                </geometry>
+                <material name="black">
+                    <color rgba="0.0 0.0 0.0 1.0"/>
+                </material>
+            </visual>
+            <!-- 碰撞特性 -->
+            <collision>
+                <geometry>
+                    <cylinder radius="0.02" length="0.02"/>
+                </geometry>
+                <material name="black">
+                    <color rgba="0.0 0.0 0.0 1.0"/>
+                </material>
+            </collision>
+            <xacro:cylinder_inertia m="0.03" r="0.02" h="0.02" />
+        </link>
+        <!-- ========== 固定laser支撑杆上 ========== -->
+        <joint name="laser_joint" type="fixed">
+            <parent link="laser_cylinder_link"/>
+            <child link="laser_link"/>
+            <!-- 位置：机器人顶部中心 (0.5/2 + 0.05/2 = 0.275) -->
+            <origin xyz="0.0 0.0 0.05" rpy="0.0 0.0 0.0"/>
+        </joint>
+        <!-- ========== 固定laser支撑杆到机器人顶部 ========== -->
+        <joint name="laser_cylinder_joint" type="fixed">
+            <parent link="base_link"/>
+            <child link="laser_cylinder_link"/>
+            <!-- 位置：机器人顶部中心 (0.5/2 + 0.05/2 = 0.275) -->
+            <origin xyz="${xyz}" rpy="0.0 0.0 0.0"/>
+        </joint>
+        <gazebo reference="laser_cylinder_link">
+            <material>Gazebo/Black</material>
+        </gazebo>
+        <gazebo reference="laser_link">
+            <material>Gazebo/Black</material>
+        </gazebo>
+    </xacro:macro>
 </robot>
