Commit message: 仿真完成

File: src/robot_description/urdf/NaviRobot/NaviRobot.ros2_control.xacro (robot description, xacro)
@@ -1,6 +1,6 @@
 <?xml version="1.0"?>
 <robot xmlns:xacro="http://www.ros.org/wiki/xacro">
-    <xacro:macro name="NaviRbot_ros2_control">
-    <ros2_control name="NaviRbotGazeboSystem" type="system">
+    <xacro:macro name="NaviRobot_ros2_control">
+    <ros2_control name="NaviRobotGazeboSystem" type="system">
             <hardware>
                 <plugin>gazebo_ros2_control/GazeboSystem</plugin>
@@ -36,4 +36,8 @@
         <plugin filename="libgazebo_ros2_control.so" name="gazebo_ros2_control">
             <parameters>$(find robot_description)/config/robot_ros2_controller.yaml</parameters>
+            <ros>
+                <remapping>/NaviRobot_diff_drive_controller/cmd_vel_unstamped:=/cmd_vel</remapping>
+                <remapping>/NaviRobot_diff_drive_controller/odom:=/odom</remapping>
+            </ros>
         </plugin>
 </gazebo>

File: src/robot_description/urdf/NaviRobot/NaviRobot.urdf.xacro (robot description, xacro)
@@ -24,4 +24,4 @@
 <!-- <xacro:gazebo_control_plugin /> -->
 <xacro:gazebo_sensor_plugin />
-<xacro:NaviRbot_ros2_control />
+<xacro:NaviRobot_ros2_control />
 </robot>

File: src/robot_description/urdf/NaviRobot/actuator/caster.urdf.xacro (robot description, xacro)
@@ -36,6 +36,6 @@
             <mu1 value="0.0" />
             <mu2 value="0.0" />
-            <kp value="1000000000.0" />
-            <kd value="1.0" />
+            <kp value="1000000.0" />
+            <kd value="10.0" />
         </gazebo>
     </xacro:macro>

File: src/robot_description/urdf/NaviRobot/actuator/wheel.urdf.xacro (robot description, xacro)
@@ -35,8 +35,8 @@
         <gazebo reference="${wheel_name}_wheel_link">
             <material>Gazebo/Black</material>
-            <mu1 value="20.0" />
-            <mu2 value="20.0" />
-            <kp value="1000000000.0" />
-            <kd value="1.0" />
+            <mu1 value="50.0" />
+            <mu2 value="50.0" />
+            <kp value="1000000.0" />
+            <kd value="10.0" />
         </gazebo>
     </xacro:macro>
