Commit message: 建图

File: src/robot_description/urdf/NaviRobot/actuator/caster.urdf.xacro (robot description, xacro)
@@ -36,6 +36,6 @@
             <mu1 value="0.0" />
             <mu2 value="0.0" />
-            <kp value="1000000.0" />
-            <kd value="10.0" />
+            <kp value="1000000000.0" />
+            <kd value="1.0" />
         </gazebo>
     </xacro:macro>

File: src/robot_description/urdf/NaviRobot/actuator/wheel.urdf.xacro (robot description, xacro)
@@ -35,8 +35,8 @@
         <gazebo reference="${wheel_name}_wheel_link">
             <material>Gazebo/Black</material>
-            <mu1 value="50.0" />
-            <mu2 value="50.0" />
-            <kp value="1000000.0" />
-            <kd value="10.0" />
+            <mu1 value="20.0" />
+            <mu2 value="20.0" />
+            <kp value="1000000000.0" />
+            <kd value="1.0" />
         </gazebo>
     </xacro:macro>

File: src/robot_description/urdf/NaviRobot/plugins/gazebo_sensor_plugin.xacro (robot description, xacro)
@@ -14,5 +14,5 @@
                 <always_on>true</always_on>
                 <visualize>true</visualize>
-                <update_rate>5</update_rate>
+                <update_rate>30</update_rate>
                 <pose>0 0 0 0 0 0</pose>
 								<!-- 激光传感器配置 -->
@@ -34,12 +34,13 @@
                     </range>
                     <!-- 设置噪声 -->
-                    <noise>
+                    <!-- <noise>
                         <type>gaussian</type>
                         <mean>0.0</mean>
                         <stddev>0.01</stddev>
-                    </noise>
+                    </noise> -->
                 </ray>
             </sensor>
         </gazebo>
+    </xacro:macro>
 <gazebo reference="imu_link">
     <sensor name="imu_sensor" type="imu">
@@ -54,5 +55,5 @@
         <always_on>true</always_on>
         <!-- 六轴噪声设置 -->
-        <imu>
+        <!-- <imu>
             <angular_velocity>
                 <x>
@@ -107,8 +108,7 @@
                 </z>
             </linear_acceleration>
-        </imu>
+        </imu> -->
     </sensor>
 </gazebo>
-    </xacro:macro>
 <gazebo reference="camera_link">
     <sensor type="depth" name="camera_sensor">
